Commit message: setup lidar

File: urdf/robot.urdf.xacro (robot description, xacro)
@@ -5,5 +5,5 @@
     <visual>
       <geometry>
-        <box size="0.5 0.3 0.1"/>
+        <box size="0.8 0.5 0.2"/>
       </geometry>
       <material name="blue">
@@ -13,5 +13,5 @@
     <collision>
       <geometry>
-        <box size="0.5 0.3 0.1"/>
+        <box size="0.8 0.5 0.2"/>
       </geometry>
     </collision>
@@ -22,9 +22,9 @@
   </link>
   <!-- Wheel macro -->
-  <xacro:macro name="wheel" params="prefix y">
+  <xacro:macro name="wheel" params="prefix y x">
     <joint name="${prefix}_wheel_joint" type="continuous">
       <parent link="base_link"/>
       <child link="${prefix}_wheel"/>
-      <origin xyz="0 ${y} 0" rpy="1.57 0 0"/>
+      <origin xyz="${x} ${y} 0" rpy="1.57 0 0"/>
       <axis xyz="0 0 1"/>
     </joint>
@@ -32,5 +32,5 @@
       <visual>
         <geometry>
-          <cylinder radius="0.1" length="0.05"/>
+          <cylinder radius="0.12" length="0.05"/>
         </geometry>
         <material name="black">
@@ -40,5 +40,5 @@
       <collision>
         <geometry>
-          <cylinder radius="0.1" length="0.05"/>
+          <cylinder radius="0.12" length="0.05"/>
         </geometry>
       </collision>
@@ -50,11 +50,11 @@
   </xacro:macro>
   <!-- Left and right wheels -->
-  <xacro:wheel prefix="left" y="0.2"/>
-  <xacro:wheel prefix="right" y="-0.2"/>
+  <xacro:wheel prefix="left" y="0.3" x="0"/>
+  <xacro:wheel prefix="right" y="-0.3" x="0"/>
   <!-- Lidar sensor -->
   <joint name="lidar_joint" type="fixed">
     <parent link="base_link"/>
     <child link="lidar_link"/>
-    <origin xyz="0.2 0 0.1"/>
+    <origin xyz="0 0 0.2"/>
   </joint>
   <link name="lidar_link">
